File: Eletro/Number Of Complete Cycles/HW/PCB/SolidStateRelay/SolidStateRelay.kicad_sch (KiCad schematic)
At the start: 13 parts, among them J1 KRE_02, Q1 BT138-600, U1 MOC3020M

Commit message: PCB update
Parts:
- removed Atuador1: ~, Connector_PinHeader_2.54mm:PinHeader_1x02_P2.54mm_Vertical, symbol Connector:Conn_01x02_Pin
- removed Sensor1: ~, Connector_Molex:Molex_KK-396_A-41792-0002_1x02_P3.96mm_Horizontal, symbol Connector:Conn_01x02_Pin
- added J2: Conn_01x05_Pin, Connector_JST:JST_EH_S5B-EH_1x05_P2.50mm_Horizontal, symbol Connector:Conn_01x05_Pin
- C1, C2: footprint Capacitor_THT:C_Disc_D7.0mm_W2.5mm_P5.00mm -> Capacitor_THT:C_Rect_L9.0mm_W3.3mm_P7.50mm_MKT
Connections:
- net at C1.2, C2.2, Q1.1 (A1): now also J1.1; no longer J1.2
- net at R5.1, SenseRead1.2 (Pin_2): now also J2.4 (Pin_4)
- net +5V: now reaches R5.2
- net +5V: now also J2.2 (Pin_2); no longer U1.2
- net at Q1.2 (A2), R2.2, R3.2: now also J1.2; no longer J1.1
- net GND: now reaches SenseRead1.1 (Pin_1)
- net GND: now also U1.2, J2.3 (Pin_3)
- net at R4.1: now also J2.1 (Pin_1)
Other:
- moved on the sheet: R5, SenseRead1

Commit message: PCB update
Parts:
- renumbered SenseRead1 to Sensor
Changed lines of the file:
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@@
   (symbol (lib_id "Connector:Conn_01x02_Pin") (at 29.21 67.31 0) (unit 1)
     (in_bom yes) (on_board yes) (dnp no) (fields_autoplaced)
-    (property "Reference" "SenseRead1" (at 29.845 66.04 0)
+    (property "Reference" "Sensor" (at 29.845 66.04 0)
       (effects (font (size 1.27 1.27)))
     )
@@
       (project "SolidStateRelay"
         (path "/400f0e6e-7eca-462d-89bc-713ac3ba06f4"
-          (reference "SenseRead1") (unit 1)
+          (reference "Sensor") (unit 1)
         )
       )
